Commit message: update

File: rb_description/urdf/rb5.urdf (robot description, URDF)
Before this commit: robot rb5, 12 links, 11 joints
Links:
- link Body_Base: geometry collision mesh filename=package://rb_description/meshes/rb5/collision/_1_base.stl scale=0.001 0.001 0.001; visual mesh filename=package://rb_description/meshes/rb5/visual/_1_base.dae
- link Body_Module_1: geometry collision mesh filename=package://rb_description/meshes/rb5/collision/_2_module_1.s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 scale=0.001 0.001 0.001; visual mesh filename=package://rb_description/meshes/rb5/visual/_2_module_1.dae
- link Body_Module_2: geometry collision mesh filename=package://rb_description/meshes/rb5/collision/_3_module_2.s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 scale=0.001 0.001 0.001; visual mesh filename=package://rb_description/meshes/rb5/visual/_3_module_2.dae
- link Body_Module_3: geometry collision mesh filename=package://rb_description/meshes/rb5/collision/_5_module_3.s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 scale=0.001 0.001 0.001; visual mesh filename=package://rb_description/meshes/rb5/visual/_5_module_3.dae
- link Body_Module_4: geometry collision mesh filename=package://rb_description/meshes/rb5/collision/_8_module_4.s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 scale=0.001 0.001 0.001; visual mesh filename=package://rb_description/meshes/rb5/visual/_8_module_4.dae
- link Body_Module_5: geometry collision mesh filename=package://rb_description/meshes/rb5/collision/_9_module_5.s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 scale=0.001 0.001 0.001; visual mesh filename=package://rb_description/meshes/rb5/visual/_9_module_5.dae
- link Body_Module_6: geometry collision mesh filename=package://rb_description/meshes/rb5/collision/_10_module_6.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 scale=0.001 0.001 0.001; visual mesh filename=package://rb_description/meshes/rb5/visual/_10_module_6.dae
- link Body_Module_Dummy: geometry collision mesh filename=package://rb_description/meshes/rb5/collision/_6_module_dum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 scale=0.001 0.001 0.001; visual mesh filename=package://rb_description/meshes/rb5/visual/_6_module_dummy.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
- link Body_Pipe_1: geometry collision mesh filename=package://rb_description/meshes/rb5/collision/_4_pipe_1.stl scale=0.001 0.001 0.001; visual mesh filename=package://rb_description/meshes/rb5/visual/_4_pipe_1.dae
- link Body_Pipe_2: geometry collision mesh filename=package://rb_description/meshes/rb5/collision/_7_pipe_2.stl scale=0.001 0.001 0.001; visual mesh filename=package://rb_description/meshes/rb5/visual/_7_pipe_2.dae
- link Body_Tool_Flange: geometry collision mesh filename=package://rb_description/meshes/rb5/collision/_11_tool_flan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 scale=0.001 0.001 0.001; visual mesh filename=package://rb_description/meshes/rb5/visual/_11_tool_flange.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
